File: 4-HCloverMedallion.brd (EAGLE design)
At the start: 50.8 x 76.2 mm, 25 parts, among them J1 ICSP, U1 TINY85-20-DIP

Commit message: updating files
Parts:
- U$2: value 4H-LOGO14 -> (none)
Changed lines of the file:
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@@
 <attribute name="NAME" x="25.4" y="18.7325" size="1.27" layer="25" ratio="10" align="top-center"/>
 </element>
-<element name="U$2" library="4h" package="4H_LOGO_14" value="4H-LOGO14" x="25.4" y="50.8"/>
+<element name="U$2" library="4h" package="4H_LOGO_14" value="" x="25.4" y="50.8"/>
 </elements>
 <signals>
